File: Hardware/Qwiic_Shield_for_Teensy_Extended.brd (EAGLE design)
At the start: 17.8 x 61 mm, 40 parts, among them J1 TEENSY_EXTENDED, J2 QWIIC_RA, J3 QWIIC_RA, J4 QWIIC_Vertical, J5 QWIIC_Vertical, J6 ALT PWR

Commit message: checklist run post design review
-adjusted values for better assembly sheet
Parts:
- S1: value (none) -> SMD_5.2MM
Changed lines of the file:
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@@
 <drawing>
 <settings>
-<setting alwaysvectorfont="no"/>
+<setting alwaysvectorfont="yes"/>
 <setting verticaltext="up"/>
 </settings>
@@
 <layer number="45" name="Holes" color="7" fill="1" visible="yes" active="yes"/>
 <layer number="46" name="Milling" color="3" fill="1" visible="no" active="yes"/>
-<layer number="47" name="Measures" color="7" fill="1" visible="yes" active="yes"/>
+<layer number="47" name="Measures" color="7" fill="1" visible="no" active="yes"/>
 <layer number="48" name="Document" color="7" fill="1" visible="no" active="yes"/>
 <layer number="49" name="Reference" color="7" fill="1" visible="yes" active="yes"/>
@@
 <attribute name="NAME" x="7.493" y="2.921" size="0.6096" layer="25" font="vector" ratio="20"/>
 <attribute name="PROD_ID" value="CONN-13694" x="8.89" y="5.08" size="1.778" layer="27" display="off"/>
-<attribute name="VALUE" x="7.239" y="1.778" size="0.6096" layer="27" font="vector" ratio="20"/>
+<attribute name="VALUE" x="6.985" y="0.889" size="0.6096" layer="27" font="vector" ratio="20"/>
 </element>
 <element name="J3" library="SparkFun-Connectors" package="JST04_1MM_RA" value="QWIIC_RA" x="8.89" y="55.88" smashed="yes" rot="R180">
 <attribute name="NAME" x="10.287" y="58.039" size="0.6096" layer="25" font="vector" ratio="20" rot="R180"/>
 <attribute name="PROD_ID" value="CONN-13694" x="8.89" y="55.88" size="1.778" layer="27" rot="R180" display="off"/>
-<attribute name="VALUE" x="10.541" y="59.182" size="0.6096" layer="27" font="vector" ratio="20" rot="R180"/>
+<attribute name="VALUE" x="10.6934" y="60.0964" size="0.6096" layer="27" font="vector" ratio="20" rot="R180"/>
 </element>
 <element name="J5" library="SparkFun-Connectors" package="JST04_1MM_VERT" value="QWIIC_Vertical" x="8.89" y="53.34" smashed="yes" rot="R180">
 <attribute name="NAME" x="8.874" y="48.77366875" size="0.6096" layer="25" rot="R180"/>
 <attribute name="PROD_ID" value="CONN-14483" x="8.89" y="53.34" size="1.778" layer="27" rot="R180" display="off"/>
-<attribute name="VALUE" x="8.874" y="54.63633125" size="0.6096" layer="27" rot="R180"/>
+<attribute name="VALUE" x="11.6426" y="48.84513125" size="0.6096" layer="27" font="vector" ratio="20" rot="R180"/>
 </element>
 <element name="LOGO1" library="SparkFun-Aesthetics" package="SFE_LOGO_NAME_FLAME_.1" value="SFE_LOGO_NAME_FLAME.1_INCH" x="8.89" y="35.4584" smashed="yes" rot="MR0"/>
@@
 <attribute name="NAME" x="4.8768" y="52.8066" size="0.6096" layer="25" font="vector" ratio="20" rot="R270" align="bottom-center"/>
 <attribute name="PROD_ID" value="RES-07857" x="9.1948" y="52.8066" size="1.778" layer="27" rot="R270" display="off"/>
-<attribute name="VALUE" x="3.3528" y="52.8066" size="0.6096" layer="27" font="vector" ratio="20" rot="R270" align="top-center"/>
+<attribute name="VALUE" x="3.4036" y="52.8066" size="0.6096" layer="27" font="vector" ratio="20" rot="R270" align="top-center"/>
 </element>
 <element name="R4" library="SparkFun-Resistors" package="0603" value="4.7k" x="4.0894" y="56.4642" smashed="yes" rot="R90">
 <attribute name="NAME" x="3.3274" y="56.4642" size="0.6096" layer="25" font="vector" ratio="20" rot="R90" align="bottom-center"/>
 <attribute name="PROD_ID" value="RES-07857" x="2.8194" y="52.6542" size="1.778" layer="27" rot="R90" display="off"/>
-<attribute name="VALUE" x="4.8514" y="56.4642" size="0.6096" layer="27" font="vector" ratio="20" rot="R90" align="top-center"/>
+<attribute name="VALUE" x="2.7432" y="56.515" size="0.6096" layer="27" font="vector" ratio="20" rot="R90" align="top-center"/>
 </element>
 <element name="I2C" library="SparkFun-Jumpers" package="SMT-JUMPER_3_NO_SILK" package3d_urn="urn:adsk.eagle:package:39285/1" value="JUMPER-SMT_3_NO_SILK" x="4.7752" y="54.7624" smashed="yes" rot="MR90">
@@
 <element name="J6" library="SparkFun-Connectors" package="1X02_NO_SILK" value="ALT PWR" x="8.89" y="8.89" smashed="yes" rot="R180">
 <attribute name="NAME" x="10.16" y="7.493" size="0.6096" layer="25" font="vector" ratio="20" rot="R180"/>
-<attribute name="VALUE" x="10.16" y="10.922" size="0.6096" layer="27" font="vector" ratio="20" rot="R180"/>
+<attribute name="VALUE" x="9.3218" y="7.6454" size="0.6096" layer="27" font="vector" ratio="20" rot="R180"/>
 </element>
 <element name="3V3_ISO" library="SparkFun-Jumpers" package="SMT-JUMPER_2_NC_TRACE_SILK" package3d_urn="urn:adsk.eagle:package:39281/1" value="" x="5.0038" y="3.7338" smashed="yes" rot="MR90">
@@
 <attribute name="NAME" x="7.112" y="12.7" size="0.6096" layer="25" font="vector" ratio="20" rot="R270" align="bottom-center"/>
 <attribute name="PROD_ID" value="DIO-14072" x="6.35" y="12.7" size="1.778" layer="27" rot="R270" display="off"/>
-<attribute name="VALUE" x="5.588" y="12.7" size="0.6096" layer="27" font="vector" ratio="20" rot="R270" align="top-center"/>
-</element>
-<element name="S1" library="SparkFun-Switches" package="TACTILE_SWITCH_SMD_5.2MM" value="" x="8.89" y="41.91" smashed="yes">
+<attribute name="VALUE" x="5.4102" y="12.7254" size="0.6096" layer="27" font="vector" ratio="20" rot="R270" align="top-center"/>
+</element>
+<element name="S1" library="SparkFun-Switches" package="TACTILE_SWITCH_SMD_5.2MM" value="SMD_5.2MM" x="8.89" y="41.91" smashed="yes">
 <attribute name="NAME" x="8.89" y="44.577" size="0.6096" layer="25" font="vector" ratio="20" align="bottom-center"/>
 <attribute name="PROD_ID" value="SWCH-14139" x="8.89" y="41.91" size="1.778" layer="27" display="off"/>
-<attribute name="VALUE" x="8.89" y="39.243" size="0.6096" layer="27" font="vector" ratio="20" align="top-center"/>
+<attribute name="VALUE" x="8.7376" y="45.2374" size="0.6096" layer="27" font="vector" ratio="20" align="top-center"/>
 </element>
 <element name="U$5" library="output" package="#ALT_3V3#0" value="" x="6.35" y="13.2334" smashed="yes" rot="MR90"/>
@@
 <attribute name="NAME" x="8.906" y="23.61633125" size="0.6096" layer="25"/>
 <attribute name="PROD_ID" value="CONN-14483" x="8.89" y="19.05" size="1.778" layer="27" display="off"/>
-<attribute name="VALUE" x="8.906" y="17.75366875" size="0.6096" layer="27"/>
+<attribute name="VALUE" x="5.9088" y="23.49406875" size="0.6096" layer="27" font="vector" ratio="20"/>
 </element>
 <element name="LOGO2" library="SparkFun-Aesthetics" package="SFE_LOGO_NAME_FLAME_.1" value="SFE_LOGO_NAME_FLAME.1_INCH" x="8.89" y="32.5882" smashed="yes"/>
